Commit message: Fix warning1

File: catkin_ws/src/track/urdf/autolabor_mini.urdf.xacro (robot description, xacro)
@@ -27,4 +27,10 @@
         </inertial>
     </link>
+    <!-- Add dummy link -->
+    <link name="dummy_link"/>
+    <joint name="dummy_joint" type="fixed">
+        <parent link="dummy_link"/>
+        <child link="base_link"/>
+    </joint>
     <!-- Left Wheel -->
     <link name="left_wheel">

Commit message: Fix warningKDL

File: catkin_ws/src/track/urdf/autolabor_mini.urdf.xacro (robot description, xacro)
@@ -7,4 +7,11 @@
     <xacro:property name="wheel_radius" value="0.085"/>
     <xacro:property name="wheel_width" value="0.045"/>
+    <!-- Add dummy link to fix KDL warning -->
+    <link name="base_footprint"/>
+    <joint name="base_joint" type="fixed">
+        <parent link="base_footprint"/>
+        <child link="base_link"/>
+        <origin xyz="0 0 ${wheel_radius}" rpy="0 0 0"/>
+    </joint>
     <!-- Base Link -->
     <link name="base_link">
@@ -88,5 +95,5 @@
             <wheelSeparation>${base_width}</wheelSeparation>
             <wheelDiameter>${2*wheel_radius}</wheelDiameter>
-            <robotBaseFrame>base_link</robotBaseFrame>
+            <robotBaseFrame>base_footprint</robotBaseFrame>
             <commandTopic>cmd_vel</commandTopic>
             <odometryTopic>odom</odometryTopic>
