Commit message: Fix Unreal Vision

File: catkin_ws/src/track/urdf/car.urdf.xacro (robot description, xacro)
@@ -31,3 +31,44 @@
     <!-- 其他车轮同样修改为绿色 -->
     <!-- ...existing code... -->
+    <!-- 添加相机链接 -->
+    <link name="camera_link">
+        <visual>
+            <geometry>
+                <box size="0.05 0.05 0.05"/>
+            </geometry>
+            <material name="black"/>
+        </visual>
+    </link>
+    <!-- 相机关节 -->
+    <joint name="camera_joint" type="fixed">
+        <parent link="base_link"/>
+        <child link="camera_link"/>
+        <origin xyz="0.2 0 0.1" rpy="0 0 0"/>
+    </joint>
+    <!-- 添加相机插件 -->
+    <gazebo reference="camera_link">
+        <sensor type="camera" name="camera">
+            <update_rate>30.0</update_rate>
+            <camera name="head">
+                <horizontal_fov>1.3962634</horizontal_fov>
+                <image>
+                    <width>640</width>
+                    <height>480</height>
+                    <format>R8G8B8</format>
+                </image>
+                <clip>
+                    <near>0.02</near>
+                    <far>300</far>
+                </clip>
+            </camera>
+            <plugin name="camera_controller" filename="libgazebo_ros_camera.so">
+                <alwaysOn>true</alwaysOn>
+                <updateRate>0.0</updateRate>
+                <cameraName>track_car/camera</cameraName>
+                <imageTopicName>image_raw</imageTopicName>
+                <cameraInfoTopicName>camera_info</cameraInfoTopicName>
+                <frameName>camera_link</frameName>
+            </plugin>
+        </sensor>
+    </gazebo>
 </robot>

Commit message: Fix error

File: catkin_ws/src/track/urdf/car.urdf.xacro (robot description, xacro)
@@ -1,5 +1,6 @@
 <?xml version="1.0"?>
 <robot name="car" xmlns:xacro="http://www.ros.org/wiki/xacro">
-    <!-- ...existing code... -->
+    <!-- 传入命名空间参数 -->
+    <xacro:arg name="robot_namespace" default=""/>
     <!-- 修改材质颜色 -->
     <material name="yellow">
@@ -9,5 +10,5 @@
         <color rgba="0 1 0 1"/>
     </material>
-    <!-- 车身部分 -->
+    <!-- 主体链接 -->
     <link name="base_link">
         <visual>
@@ -19,4 +20,10 @@
         <!-- ...existing code... -->
     </link>
+    <!-- 车轮链接 -->
+    <joint name="wheel_1_joint" type="continuous">
+        <parent link="base_link"/>
+        <child link="wheel_1"/>
+        <!-- ...existing code... -->
+    </joint>
     <!-- 车轮部分 -->
     <link name="wheel_1">

Commit message: Fix error5

File: catkin_ws/src/track/urdf/car.urdf.xacro (robot description, xacro)
@@ -12,4 +12,9 @@
     <!-- Main body link -->
     <link name="base_link">
+        <inertial>
+            <mass value="1.0"/>
+            <origin xyz="0 0 0" rpy="0 0 0"/>
+            <inertia ixx="0.0395" ixy="0" ixz="0" iyy="0.086" iyz="0" izz="0.0125"/>
+        </inertial>
         <visual>
             <geometry>
@@ -18,4 +23,9 @@
             <material name="yellow"/>
         </visual>
+        <collision>
+            <geometry>
+                <box size="0.5 0.3 0.1"/>
+            </geometry>
+        </collision>
         <!-- ...existing code... -->
     </link>
@@ -28,4 +38,9 @@
     <!-- Wheel link -->
     <link name="wheel_1">
+        <inertial>
+            <mass value="0.1"/>
+            <origin xyz="0 0 0" rpy="0 0 0"/>
+            <inertia ixx="0.000375" ixy="0" ixz="0" iyy="0.000375" iyz="0" izz="0.00072"/>
+        </inertial>
         <visual>
             <geometry>
@@ -34,4 +49,9 @@
             <material name="green"/>
         </visual>
+        <collision>
+            <geometry>
+                <cylinder radius="0.06" length="0.04"/>
+            </geometry>
+        </collision>
         <!-- ...existing code... -->
     </link>
@@ -79,3 +99,24 @@
         </sensor>
     </gazebo>
+    <!-- Add Gazebo plugins for differential drive -->
+    <gazebo>
+        <plugin name="differential_drive_controller" filename="libgazebo_ros_diff_drive.so">
+            <leftJoint>wheel_1_joint</leftJoint>
+            <rightJoint>wheel_2_joint</rightJoint>
+            <robotNamespace>$(arg robot_namespace)</robotNamespace>
+            <wheelSeparation>0.3</wheelSeparation>
+            <wheelDiameter>0.12</wheelDiameter>
+            <commandTopic>cmd_vel</commandTopic>
+            <odometryTopic>odom</odometryTopic>
+            <odometryFrame>odom</odometryFrame>
+            <robotBaseFrame>base_link</robotBaseFrame>
+            <publishWheelTF>false</publishWheelTF>
+            <publishOdomTF>true</publishOdomTF>
+            <publishWheelJointState>false</publishWheelJointState>
+            <wheelAcceleration>1.0</wheelAcceleration>
+            <wheelTorque>20</wheelTorque>
+            <odometrySource>world</odometrySource>
+            <updateRate>30</updateRate>
+        </plugin>
+    </gazebo>
 </robot>

Commit message: Fix error6

File: catkin_ws/src/track/urdf/car.urdf.xacro (robot description, xacro)
@@ -9,4 +9,7 @@
     <material name="green">
         <color rgba="0 1 0 1"/>
+    </material>
+    <material name="black">
+        <color rgba="0 0 0 1"/>
     </material>
     <!-- Main body link -->
@@ -21,5 +24,10 @@
                 <box size="0.5 0.3 0.1"/>
             </geometry>
-            <material name="yellow"/>
+            <xacro:if value="${robot_namespace == 'target_car'}">
+                <material name="green"/>
+            </xacro:if>
+            <xacro:if value="${robot_namespace == 'track_car'}">
+                <material name="yellow"/>
+            </xacro:if>
         </visual>
         <collision>
@@ -47,5 +55,5 @@
                 <cylinder radius="0.06" length="0.04"/>
             </geometry>
-            <material name="green"/>
+            <material name="black"/>
         </visual>
         <collision>
@@ -55,4 +63,30 @@
         </collision>
         <!-- ...existing code... -->
+    </link>
+    <!-- 添加右轮关节 -->
+    <joint name="wheel_2_joint" type="continuous">
+        <parent link="base_link"/>
+        <child link="wheel_2"/>
+        <origin xyz="0 -0.15 -0.05" rpy="0 0 0"/>
+        <axis xyz="0 1 0"/>
+    </joint>
+    <!-- 添加右轮连杆 -->
+    <link name="wheel_2">
+        <inertial>
+            <mass value="0.1"/>
+            <origin xyz="0 0 0" rpy="0 0 0"/>
+            <inertia ixx="0.000375" ixy="0" ixz="0" iyy="0.000375" iyz="0" izz="0.00072"/>
+        </inertial>
+        <visual>
+            <geometry>
+                <cylinder radius="0.06" length="0.04"/>
+            </geometry>
+            <material name="black"/>
+        </visual>
+        <collision>
+            <geometry>
+                <cylinder radius="0.06" length="0.04"/>
+            </geometry>
+        </collision>
     </link>
     <!-- Other wheels are also green -->

Commit message: Fix error8

File: catkin_ws/src/track/urdf/car.urdf.xacro (robot description, xacro)
@@ -2,5 +2,5 @@
 <robot name="car" xmlns:xacro="http://www.ros.org/wiki/xacro">
     <!-- Robot namespace parameter -->
-    <xacro:arg name="robot_namespace" default=""/>
+    <xacro:property name="robot_type" value="track_car"/>
     <!-- Materials -->
     <material name="yellow">
@@ -24,10 +24,6 @@
                 <box size="0.5 0.3 0.1"/>
             </geometry>
-            <xacro:if value="${robot_namespace == 'target_car'}">
-                <material name="green"/>
-            </xacro:if>
-            <xacro:if value="${robot_namespace == 'track_car'}">
-                <material name="yellow"/>
-            </xacro:if>
+            <material name="yellow" if="$(eval robot_type == 'track_car')"/>
+            <material name="green" if="$(eval robot_type == 'target_car')"/>
         </visual>
         <collision>

Commit message: Fix error9

File: catkin_ws/src/track/urdf/car.urdf.xacro (robot description, xacro)
@@ -1,6 +1,6 @@
 <?xml version="1.0" encoding="UTF-8"?>
 <robot name="car" xmlns:xacro="http://www.ros.org/wiki/xacro">
-    <!-- Robot namespace parameter -->
-    <xacro:property name="robot_type" value="track_car"/>
+    <!-- Robot type parameter -->
+    <xacro:arg name="robot_type" default="track_car"/>
     <!-- Materials -->
     <material name="yellow">
@@ -24,6 +24,10 @@
                 <box size="0.5 0.3 0.1"/>
             </geometry>
-            <material name="yellow" if="$(eval robot_type == 'track_car')"/>
-            <material name="green" if="$(eval robot_type == 'target_car')"/>
+            <xacro:if value="$(arg robot_type) == 'track_car'">
+                <material name="yellow"/>
+            </xacro:if>
+            <xacro:if value="$(arg robot_type) == 'target_car'">
+                <material name="green"/>
+            </xacro:if>
         </visual>
         <collision>

Commit message: Fix error13

File: catkin_ws/src/track/urdf/car.urdf.xacro (robot description, xacro)
@@ -24,10 +24,6 @@
                 <box size="0.5 0.3 0.1"/>
             </geometry>
-            <xacro:if value="${'$(arg robot_type)' == 'track_car'}">
-                <material name="yellow"/>
-            </xacro:if>
-            <xacro:if value="${'$(arg robot_type)' == 'target_car'}">
-                <material name="green"/>
-            </xacro:if>
+            <material name="yellow" if="$(eval robot_type == 'track_car')"/>
+            <material name="green" if="$(eval robot_type == 'target_car')"/>
         </visual>
         <collision>

Commit message: Fix error14

File: catkin_ws/src/track/urdf/car.urdf.xacro (robot description, xacro)
@@ -13,4 +13,11 @@
         <color rgba="0 0 0 1"/>
     </material>
+    <!-- Add virtual root link -->
+    <link name="virtual_root"/>
+    <joint name="virtual_joint" type="fixed">
+        <parent link="virtual_root"/>
+        <child link="base_link"/>
+        <origin xyz="0 0 0" rpy="0 0 0"/>
+    </joint>
     <!-- Main body link -->
     <link name="base_link">
@@ -41,12 +48,4 @@
     </joint>
     <!-- Wheel link -->
-    <link name="wheel_1">
-        <inertial>
-            <mass value="0.1"/>
-            <origin xyz="0 0 0" rpy="0 0 0"/>
-            <inertia ixx="0.000375" ixy="0" ixz="0" iyy="0.000375" iyz="0" izz="0.00072"/>
-        </inertial>
-        <visual>
-            <geometry>
                 <cylinder radius="0.06" length="0.04"/>
             </geometry>
@@ -60,5 +59,5 @@
         <!-- ...existing code... -->
     </link>
-    <!-- 添加右轮关节 -->
+    <!-- Right wheel -->
     <joint name="wheel_2_joint" type="continuous">
         <parent link="base_link"/>
@@ -67,5 +66,5 @@
         <axis xyz="0 1 0"/>
     </joint>
-    <!-- 添加右轮连杆 -->
+    <!-- Right wheel link -->
     <link name="wheel_2">
         <inertial>
@@ -151,2 +150,10 @@
     </gazebo>
 </robot>
+            <publishWheelJointState>false</publishWheelJointState>
+            <wheelAcceleration>1.0</wheelAcceleration>
+            <wheelTorque>20</wheelTorque>
+            <odometrySource>world</odometrySource>
+            <updateRate>30</updateRate>
+        </plugin>
+    </gazebo>
+</robot>

Commit message: Fix error15

File: catkin_ws/src/track/urdf/car.urdf.xacro (robot description, xacro)
@@ -39,13 +39,20 @@
             </geometry>
         </collision>
-        <!-- ...existing code... -->
     </link>
-    <!-- Wheel joint -->
+    <!-- Left wheel -->
     <joint name="wheel_1_joint" type="continuous">
         <parent link="base_link"/>
         <child link="wheel_1"/>
-        <!-- ...existing code... -->
+        <origin xyz="0 0.15 -0.05" rpy="0 0 0"/>
+        <axis xyz="0 1 0"/>
     </joint>
-    <!-- Wheel link -->
+    <link name="wheel_1">
+        <inertial>
+            <mass value="0.1"/>
+            <origin xyz="0 0 0" rpy="0 0 0"/>
+            <inertia ixx="0.000375" ixy="0" ixz="0" iyy="0.000375" iyz="0" izz="0.00072"/>
+        </inertial>
+        <visual>
+            <geometry>
                 <cylinder radius="0.06" length="0.04"/>
             </geometry>
@@ -57,5 +64,4 @@
             </geometry>
         </collision>
-        <!-- ...existing code... -->
     </link>
     <!-- Right wheel -->
@@ -66,5 +72,4 @@
         <axis xyz="0 1 0"/>
     </joint>
-    <!-- Right wheel link -->
     <link name="wheel_2">
         <inertial>
@@ -85,7 +90,5 @@
         </collision>
     </link>
-    <!-- Other wheels are also green -->
-    <!-- ...existing code... -->
-    <!-- Camera link -->
+    <!-- Camera link and joint -->
     <link name="camera_link">
         <visual>
@@ -96,5 +99,4 @@
         </visual>
     </link>
-    <!-- Camera joint -->
     <joint name="camera_joint" type="fixed">
         <parent link="base_link"/>
@@ -102,5 +104,5 @@
         <origin xyz="0.2 0 0.1" rpy="0 0 0"/>
     </joint>
-    <!-- Camera plugin -->
+    <!-- Gazebo plugins -->
     <gazebo reference="camera_link">
         <sensor type="camera" name="camera">
@@ -128,5 +130,4 @@
         </sensor>
     </gazebo>
-    <!-- Add Gazebo plugins for differential drive -->
     <gazebo>
         <plugin name="differential_drive_controller" filename="libgazebo_ros_diff_drive.so">
@@ -150,10 +151,2 @@
     </gazebo>
 </robot>
-            <publishWheelJointState>false</publishWheelJointState>
-            <wheelAcceleration>1.0</wheelAcceleration>
-            <wheelTorque>20</wheelTorque>
-            <odometrySource>world</odometrySource>
-            <updateRate>30</updateRate>
-        </plugin>
-    </gazebo>
-</robot>

Commit message: Fix error19

File: catkin_ws/src/track/urdf/car.urdf.xacro (robot description, xacro)
@@ -1,4 +1,6 @@
 <?xml version="1.0" encoding="UTF-8"?>
 <robot name="car" xmlns:xacro="http://www.ros.org/wiki/xacro">
+    <!-- 包含其他xacro文件 -->
+    <xacro:include filename="$(find track)/urdf/common.xacro" />
     <!-- Robot type parameter -->
     <xacro:arg name="robot_type" default="track_car"/>
@@ -20,4 +22,14 @@
         <origin xyz="0 0 0" rpy="0 0 0"/>
     </joint>
+    <!-- 底盘 -->
+    <xacro:property name="base_radius" value="0.20"/>
+    <xacro:property name="base_length" value="0.30"/>
+    <xacro:property name="base_height" value="0.15"/>
+    <!-- 车轮参数 -->
+    <xacro:property name="wheel_radius" value="0.06"/>
+    <xacro:property name="wheel_width" value="0.04"/>
+    <xacro:property name="wheel_ygap" value="0.20"/>
+    <xacro:property name="wheel_zoff" value="0.05"/>
+    <xacro:property name="wheel_xoff" value="0.12"/>
     <!-- Main body link -->
     <link name="base_link">
@@ -29,5 +41,5 @@
         <visual>
             <geometry>
-                <box size="0.5 0.3 0.1"/>
+                <box size="${base_length} ${base_radius*2} ${base_height}"/>
             </geometry>
             <material name="yellow" if="$(eval robot_type == 'track_car')"/>
@@ -36,58 +48,38 @@
         <collision>
             <geometry>
-                <box size="0.5 0.3 0.1"/>
+                <box size="${base_length} ${base_radius*2} ${base_height}"/>
             </geometry>
         </collision>
     </link>
-    <!-- Left wheel -->
-    <joint name="wheel_1_joint" type="continuous">
-        <parent link="base_link"/>
-        <child link="wheel_1"/>
-        <origin xyz="0 0.15 -0.05" rpy="0 0 0"/>
-        <axis xyz="0 1 0"/>
-    </joint>
-    <link name="wheel_1">
-        <inertial>
-            <mass value="0.1"/>
-            <origin xyz="0 0 0" rpy="0 0 0"/>
-            <inertia ixx="0.000375" ixy="0" ixz="0" iyy="0.000375" iyz="0" izz="0.00072"/>
-        </inertial>
-        <visual>
-            <geometry>
-                <cylinder radius="0.06" length="0.04"/>
-            </geometry>
-            <material name="black"/>
-        </visual>
-        <collision>
-            <geometry>
-                <cylinder radius="0.06" length="0.04"/>
-            </geometry>
-        </collision>
-    </link>
-    <!-- Right wheel -->
-    <joint name="wheel_2_joint" type="continuous">
-        <parent link="base_link"/>
-        <child link="wheel_2"/>
-        <origin xyz="0 -0.15 -0.05" rpy="0 0 0"/>
-        <axis xyz="0 1 0"/>
-    </joint>
-    <link name="wheel_2">
-        <inertial>
-            <mass value="0.1"/>
-            <origin xyz="0 0 0" rpy="0 0 0"/>
-            <inertia ixx="0.000375" ixy="0" ixz="0" iyy="0.000375" iyz="0" izz="0.00072"/>
-        </inertial>
-        <visual>
-            <geometry>
-                <cylinder radius="0.06" length="0.04"/>
-            </geometry>
-            <material name="black"/>
-        </visual>
-        <collision>
-            <geometry>
-                <cylinder radius="0.06" length="0.04"/>
-            </geometry>
-        </collision>
-    </link>
+    <!-- 四个车轮宏定义 -->
+    <xacro:macro name="wheel" params="prefix x_reflect y_reflect">
+        <joint name="${prefix}_wheel_joint" type="continuous">
+            <parent link="base_link"/>
+            <child link="${prefix}_wheel"/>
+            <origin xyz="${wheel_xoff * x_reflect} ${wheel_ygap/2 * y_reflect} ${-wheel_zoff}" rpy="0 0 0"/>
+            <axis xyz="0 1 0"/>
+        </joint>
+        <link name="${prefix}_wheel">
+            <visual>
+                <geometry>
+                    <cylinder radius="${wheel_radius}" length="${wheel_width}"/>
+                </geometry>
+                <material name="black"/>
+                <origin xyz="0 0 0" rpy="${pi/2} 0 0"/>
+            </visual>
+            <collision>
+                <geometry>
+                    <cylinder radius="${wheel_radius}" length="${wheel_width}"/>
+                </geometry>
+                <origin xyz="0 0 0" rpy="${pi/2} 0 0"/>
+            </collision>
+            <xacro:default_inertial mass="1"/>
+        </link>
+    </xacro:macro>
+    <!-- 添加四个车轮 -->
+    <xacro:wheel prefix="front_right" x_reflect="1" y_reflect="-1" />
+    <xacro:wheel prefix="front_left" x_reflect="1" y_reflect="1" />
+    <xacro:wheel prefix="rear_right" x_reflect="-1" y_reflect="-1" />
+    <xacro:wheel prefix="rear_left" x_reflect="-1" y_reflect="1" />
     <!-- Camera link and joint -->
     <link name="camera_link">

Commit message: Fix error23

File: catkin_ws/src/track/urdf/car.urdf.xacro (robot description, xacro)
@@ -22,9 +22,9 @@
         <origin xyz="0 0 0" rpy="0 0 0"/>
     </joint>
-    <!-- 底盘 -->
+    <!-- Base parameters -->
     <xacro:property name="base_radius" value="0.20"/>
     <xacro:property name="base_length" value="0.30"/>
     <xacro:property name="base_height" value="0.15"/>
-    <!-- 车轮参数 -->
+    <!-- Wheel parameters -->
     <xacro:property name="wheel_radius" value="0.06"/>
     <xacro:property name="wheel_width" value="0.04"/>

File: catkin_ws/src/track/urdf/common.xacro (robot description, xacro)
@@ -1,7 +1,7 @@
 <?xml version="1.0"?>
 <robot xmlns:xacro="http://www.ros.org/wiki/xacro">
-    <!-- 常量定义 -->
-    <xacro:property name="pi" value="3.1415926"/>
-    <!-- 默认惯性参数宏 -->
+    <!-- Constants -->
+    <!-- pi is already defined in xacro, no need to redefine -->
+    <!-- Default inertial macro -->
     <xacro:macro name="default_inertial" params="mass">
         <inertial>
@@ -14,5 +14,5 @@
         </inertial>
     </xacro:macro>
-    <!-- 材质定义 -->
+    <!-- Materials -->
     <material name="white">
         <color rgba="1 1 1 1"/>

Commit message: 增强目标跟踪功能，调整掩码范围以适应Gazebo中的颜色，添加深度信息处理和控制逻辑，提升跟踪准确性和稳定性

File: catkin_ws/src/track/urdf/car.urdf.xacro (robot description, xacro)
@@ -96,5 +96,5 @@
     <!-- Gazebo plugins -->
     <gazebo reference="camera_link">
-        <sensor type="camera" name="camera">
+        <sensor type="depth" name="camera">
             <update_rate>30.0</update_rate>
             <camera name="head">
@@ -109,6 +109,12 @@
                     <far>300</far>
                 </clip>
+                <noise>
+                    <type>gaussian</type>
+                    <mean>0.0</mean>
+                    <stddev>0.007</stddev>
+                </noise>
             </camera>
-            <plugin name="camera_controller" filename="libgazebo_ros_camera.so">
+            <plugin name="kinect_camera_controller" filename="libgazebo_ros_openni_kinect.so">
+                <baseline>0.2</baseline>
                 <alwaysOn>true</alwaysOn>
                 <updateRate>30.0</updateRate>
@@ -116,13 +122,18 @@
                 <imageTopicName>image_raw</imageTopicName>
                 <cameraInfoTopicName>camera_info</cameraInfoTopicName>
+                <depthImageTopicName>depth/image_raw</depthImageTopicName>
+                <depthImageInfoTopicName>depth/camera_info</depthImageInfoTopicName>
+                <pointCloudTopicName>depth/points</pointCloudTopicName>
                 <frameName>camera_link</frameName>
-                <hackBaseline>0.07</hackBaseline>
-                <distortionK1>0.0</distortionK1>
-                <distortionK2>0.0</distortionK2>
-                <distortionK3>0.0</distortionK3>
-                <distortionT1>0.0</distortionT1>
-                <distortionT2>0.0</distortionT2>
+                <pointCloudCutoff>0.5</pointCloudCutoff>
+                <pointCloudCutoffMax>3.0</pointCloudCutoffMax>
+                <distortionK1>0.00000001</distortionK1>
+                <distortionK2>0.00000001</distortionK2>
+                <distortionK3>0.00000001</distortionK3>
+                <distortionT1>0.00000001</distortionT1>
+                <distortionT2>0.00000001</distortionT2>
             </plugin>
         </sensor>
+        <material>Gazebo/Black</material>
     </gazebo>
     <!-- Modify differential drive plugin configuration -->
@@ -147,3 +158,32 @@
         </plugin>
     </gazebo>
+    <!-- Gazebo Materials -->
+    <gazebo reference="base_link">
+        <material>Gazebo/Yellow</material>
+        <plugin name="base_controller" filename="libgazebo_ros_control.so">
+            <robotNamespace>$(arg robot_type)</robotNamespace>
+        </plugin>
+    </gazebo>
+    <!-- Add color for wheels -->
+    <gazebo reference="front_right_wheel">
+        <material>Gazebo/Black</material>
+    </gazebo>
+    <gazebo reference="front_left_wheel">
+        <material>Gazebo/Black</material>
+    </gazebo>
+    <gazebo reference="rear_right_wheel">
+        <material>Gazebo/Black</material>
+    </gazebo>
+    <gazebo reference="rear_left_wheel">
+        <material>Gazebo/Black</material>
+    </gazebo>
+    <!-- Conditional material for base_link based on robot type -->
+    <gazebo reference="base_link">
+        <xacro:if value="$(eval robot_type == 'track_car')">
+            <material>Gazebo/Yellow</material>
+        </xacro:if>
+        <xacro:if value="$(eval robot_type == 'target_car')">
+            <material>Gazebo/Green</material>
+        </xacro:if>
+    </gazebo>
 </robot>
